File: buck.kicad_sch (KiCad schematic)
At the start: 9 parts, among them J7 XT60-M, U1 LMR51430

Commit message: final changes
Parts:
- renumbered C8 to C20, C9 to C21, C10 to C22, C11 to C23, J7 to J4, R2 to R17, R3 to R18
Changed lines of the file:
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@@
 		(dnp no)
 		(fields_autoplaced yes)
-		(property "Reference" "R2"
+		(property "Reference" "R17"
 			(at 175.26 97.7899 90)
 			(effects
@@
 			(project "harm_drone"
 				(path "/5ce3566e-4e0f-420e-9b0d-3952cd3c63fd/9be4028a-d272-4251-aa6b-aa28299b7605"
-					(reference "R2")
+					(reference "R17")
 					(unit 1)
 				)
@@
 		(dnp no)
 		(fields_autoplaced yes)
-		(property "Reference" "C11"
+		(property "Reference" "C23"
 			(at 205.74 106.6799 90)
 			(effects
@@
 			(project "harm_drone"
 				(path "/5ce3566e-4e0f-420e-9b0d-3952cd3c63fd/9be4028a-d272-4251-aa6b-aa28299b7605"
-					(reference "C11")
+					(reference "C23")
 					(unit 1)
 				)
@@
 		(dnp no)
 		(fields_autoplaced yes)
-		(property "Reference" "J7"
+		(property "Reference" "J4"
 			(at 102.87 64.7699 90)
 			(effects
@@
 			(project ""
 				(path "/5ce3566e-4e0f-420e-9b0d-3952cd3c63fd/9be4028a-d272-4251-aa6b-aa28299b7605"
-					(reference "J7")
+					(reference "J4")
 					(unit 1)
 				)
@@
 		(dnp no)
 		(fields_autoplaced yes)
-		(property "Reference" "#PWR022"
+		(property "Reference" "#PWR024"
 			(at 115.57 115.57 0)
 			(effects
@@
 			(project "harm_drone"
 				(path "/5ce3566e-4e0f-420e-9b0d-3952cd3c63fd/9be4028a-d272-4251-aa6b-aa28299b7605"
-					(reference "#PWR022")
+					(reference "#PWR024")
 					(unit 1)
 				)
@@
 		(dnp no)
 		(fields_autoplaced yes)
-		(property "Reference" "#PWR023"
+		(property "Reference" "#PWR025"
 			(at 186.69 139.7 0)
 			(effects
@@
 			(project "harm_drone"
 				(path "/5ce3566e-4e0f-420e-9b0d-3952cd3c63fd/9be4028a-d272-4251-aa6b-aa28299b7605"
-					(reference "#PWR023")
+					(reference "#PWR025")
 					(unit 1)
 				)
@@
 		(dnp no)
 		(fields_autoplaced yes)
-		(property "Reference" "C9"
+		(property "Reference" "C21"
 			(at 135.89 76.2 0)
 			(effects
@@
 			(project "harm_drone"
 				(path "/5ce3566e-4e0f-420e-9b0d-3952cd3c63fd/9be4028a-d272-4251-aa6b-aa28299b7605"
-					(reference "C9")
+					(reference "C21")
 					(unit 1)
 				)
@@
 		(dnp no)
 		(fields_autoplaced yes)
-		(property "Reference" "C10"
+		(property "Reference" "C22"
 			(at 190.5 106.6799 90)
 			(effects
@@
 			(project "harm_drone"
 				(path "/5ce3566e-4e0f-420e-9b0d-3952cd3c63fd/9be4028a-d272-4251-aa6b-aa28299b7605"
-					(reference "C10")
+					(reference "C22")
 					(unit 1)
 				)
@@
 		(dnp no)
 		(fields_autoplaced yes)
-		(property "Reference" "#PWR019"
+		(property "Reference" "#PWR023"
 			(at 99.06 81.28 0)
 			(effects
@@
 			(project "harm_drone"
 				(path "/5ce3566e-4e0f-420e-9b0d-3952cd3c63fd/9be4028a-d272-4251-aa6b-aa28299b7605"
-					(reference "#PWR019")
+					(reference "#PWR023")
 					(unit 1)
 				)
@@
 		(dnp no)
 		(fields_autoplaced yes)
-		(property "Reference" "C8"
+		(property "Reference" "C20"
 			(at 100.33 91.4399 90)
 			(effects
@@
 			(project "harm_drone"
 				(path "/5ce3566e-4e0f-420e-9b0d-3952cd3c63fd/9be4028a-d272-4251-aa6b-aa28299b7605"
-					(reference "C8")
+					(reference "C20")
 					(unit 1)
 				)
@@
 		(dnp no)
 		(fields_autoplaced yes)
-		(property "Reference" "R3"
+		(property "Reference" "R18"
 			(at 175.26 119.3799 90)
 			(effects
@@
 			(project "harm_drone"
 				(path "/5ce3566e-4e0f-420e-9b0d-3952cd3c63fd/9be4028a-d272-4251-aa6b-aa28299b7605"
-					(reference "R3")
-					(unit 1)
-				)
+					(reference "R18")
+					(unit 1)
+				)
